Commit message: Working velocity controller

File: rosbot_ros/src/rosbot_description/urdf/rosbot.xacro (robot description, xacro)
@@ -237,7 +237,6 @@
   <!-- Orbbec Astra RGBD Camera -->
   <joint name="astra_joint" type="continuous">
-    <axis xyz="0 0 0" rpy="0 0 0"/>
-    <limit effort="1" velocity="10"/>
-    <joint_properties damping="5.0" friction="1.0"/>
+    <axis xyz="0 0 1"/>
+    <limit effort="1" velocity="10"/>
     <origin xyz="-0.03 0 0.18" rpy="0 0 0"/>
     <parent link="body_link"/>
@@ -247,5 +246,6 @@
     <type>transmission_interface/SimpleTransmission</type>
     <actuator name="astra_motor">
-      <mechanicalReduction>1</mechanicalReduction>
+      <mechanicalInterface>1</mechanicalInterface>
+      <hardwareInterface>hardware_interface/EffortJointInterface</hardwareInterface>
     </actuator>
     <joint name="astra_joint">
